File: kicad/xy4150.sch (KiCad schematic (older format))
At the start: 219 parts, among them U1 4011, U10 7403, U11 4001, U12 4001, U13 4013, U14 4069, U15 4001, U2 4011, U3 4029, U4 4029, U5 4069, U6 4001, U7 4012, U8 4001, U9 4001

Commit message: schema fixes
Parts:
- removed J? (x12): MG, symbol Connector:Conn_01x01_Female
- removed unit 3 of U8 (x2)
- added J? (x2): Conn_01x06, symbol Connector_Generic:Conn_01x06
- added unit 3 of U8
- added unit 2 of U8
- gave numbers to parts that had none: 18
Connections:
- net GND is gone; now on net +5V: C?.1, C?.1, C?.1, C?.2, C?.2, C?.2, C?.2, C?.2, C?.2, C?.2, C?.2, C?.2, C?.2, C?.2, C?.2, C?.2, D?.2 (A), D?.2 (A), D?.2 (A), D?.2 (A), D?.2 (A), D?.2 (A), D?.2 (A), D?.2 (A), D?.2 (A), D?.2 (A), D?.2 (A), D?.2 (A), J?.1 (Pin_1), J?.1 (Pin_1), Q?.1 (E), Q?.1 (E), R16.1, R35.2, R?.2, R?.2, R?.2, R?.2, R?.2, R?.2, R?.2, R?.2, SA2.1, SA3.1, SA4.1, U10.7 (GND), U10.7 (GND), U10.7 (GND), U13.10 (R), U13.8 (S), U3.1 (PE), U3.8 (VSS), U4.1 (PE), U4.8 (VSS), U?.2 (GND), U?.4 (R), U?.7 (GND), VT?.1 (E), VT?.1 (E), VT?.1 (E), VT?.1 (E), VT?.1 (E), VT?.1 (E), VT?.1 (E), VT?.1 (E)
- net Vdd is gone; now on net +5V: U8.14 (Vdd), U8.14 (Vdd)
- net Vss is gone; now on net +5V: U8.7 (Vss), U8.7 (Vss)
- net +5V: now also R1.1, R2.1, R3.1, R4.1, U10.14 (Vcc), U10.14 (Vcc), U10.14 (Vcc), U8.1, U?.14 (Vcc), VT11.1 (E), VT5.1 (E), VT6.1 (E), VT?.1 (E), U8.14 (Vdd), U8.14 (Vdd), U8.7 (Vss), U8.7 (Vss); no longer U8.13
- net +9V: now also C?.1, JP?.2 (B), JP?.2 (B), U?.1 (IN)
- net at R4.2, SA3.2, U1.13: now also U2.9; no longer U2.8
- net at R3.2, SA4.2: now also U2.8; no longer U2.9
- net at C?.1, U13.11 (C), U2.6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: no longer C?.1, R?.2, U7.5
- net at U3.11 (Q2), U5.1, U9.9: now also U8.9
- net at U11.1, U14.5, U3.14 (Q3): now also U8.8; no longer U11.9, U8.11
- net at U6.13, U7.2: now also J?.1 (Pin_1), R7.2
- net at U11.13, U8.12: now also U8.10
- net m1-1: now reaches U11.4
- net m1-1: now also R45.1
- net m1-2: now reaches U11.11
- net m1-2: now also R48.1
- net m1-3: now reaches U11.3
- net m1-3: now also R47.1
- net m1-4: now reaches U11.10
- net m1-4: now also R46.1
- net m1-5: now reaches U12.4
- net m1-5: now also R50.1
- net m1-6: now reaches U?.11
- net m1-6: now also R49.1
- net at C?.1, R19.1, R?.1: now also U14.1; no longer U14.9
- net at C?.2, R20.1, R25.1: now also U14.13; no longer U14.11
- net at R?.2, U2.2, U7.1: no longer J?.1 (Pin_1), R7.2
- net at D?.1 (K), VT1.3 (C), VT?.3 (C): now also J?.1 (Pin_1)
- net at D?.1 (K), VT2.3 (C), VT?.3 (C): now also J?.2 (Pin_2)
- net at D?.1 (K), VT3.3 (C), VT?.3 (C): now also J?.3 (Pin_3)
- net at D?.1 (K), VT4.3 (C), VT?.3 (C): now also J?.4 (Pin_4)
- net at D?.1 (K), VT7.3 (C), VT?.3 (C): now also J?.1 (Pin_1)
- net m2-1: now reaches R?.1
- net m2-1: now also U12.10
- net at D?.1 (K), VT8.3 (C), VT?.3 (C): now also J?.2 (Pin_2)
- net m2-4: now reaches R?.1
- net m2-4: now also U15.11
- net at D?.1 (K), VT9.3 (C), VT?.3 (C): now also J?.3 (Pin_3)
- net m2-3: now reaches R?.1
- net m2-3: now also U15.10
- net at D?.1 (K), VT10.3 (C), VT?.3 (C): now also J?.4 (Pin_4)
- net m2-2: now reaches R?.1
- net m2-2: now also U12.3
- net at D?.1 (K), D?.2 (A), Q?.2 (C): now also J?.5 (Pin_5) (x2)
- net at D?.1 (K), D?.2 (A), Q?.2 (C): now also J?.6 (Pin_6) (x2)
- net m2-6: now reaches R?.1
- net m2-6: now also U15.4
- net m2-5: now reaches R?.1
- net m2-5: now also U15.3
- net Vcc: no longer names the net of J?.1 (Pin_1), R?.2, U10.10, U10.11, U10.9
- net Vcc: no longer U10.14 (Vcc), U10.14 (Vcc), U10.14 (Vcc), U?.14 (Vcc)
- new net: U11.9, U8.11
- new net: U4.11 (Q2), U5.3, U8.5, U9.5
- new net: U14.3, U15.8, U4.14 (Q3), U8.6
- new net: U4.6 (Q1), U9.2, U9.6
- new net: U5.4, U9.1
- new net: D?.2 (A), R?.1, U12.8, U15.6, U15.9, U9.4
- new net: D?.2 (A), R?.1, U12.1, U15.13, U15.2, U9.3
- new net: U12.9, U14.4
- new net: U12.2, U8.2, U8.4
- new net: U15.12, U8.3
- new net: U14.2, U15.1
- new net: U14.12, U15.5
- new net: C?.1, R?.2, U7.5
Other:
- moved on the sheet: JP?, U10A

Commit message: component library
Parts:
- removed Q? (x5): BC636, Package_TO_SOT_THT:TO-92_Inline, symbol Transistor_BJT:BC636
- removed Q? (x5), VT1, VT10, VT11, VT2, VT3, VT4, VT5, VT6, VT7, VT8, VT9, VT? (x9): BC107, Package_TO_SOT_THT:TO-18-3, symbol Transistor_BJT:BC107
- added VT, VT1, VT10, VT11, VT12, VT15, VT16, VT17, VT18, VT19, VT2, VT20, VT21, VT22, VT4, VT5, VT6, VT7, VT8, VT9, VT? (x6): KC639, Package_TO_SOT_THT:TO-92, symbol xy4150-restore:KC639
- added VT26, VT27, VT28, VT29: KD140, Package_TO_SOT_THT:TO-126-3_Vertical, symbol xy4150-restore:KD140
Connections:
- net +24V: now also VT26.1, VT27.1, VT28.1, VT29.1
- net +5V: now also VT11.1, VT12.1, VT15.1, VT16.1, VT17.1, VT18.1, VT19.1, VT20.1, VT21.1, VT22.1, VT5.1, VT6.1, VT?.1, VT?.1, VT?.3, VT?.3
- net at R?.2: now also VT?.1
- net at R32.1: now also VT?.2
- net at R33.1: now also VT?.3
- net at C?.2, D?.1 (K), R37.2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: now also VT?.1
- net at C?.1, C?.1, C?.2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: now also VT?.2
- net at C?.1, R?.1, R?.1: now also VT?.2, VT?.3
- net at R37.1: now also VT?.1, VT?.2
- net at C?.2, D?.2 (A), R38.1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: now also VT?.1
- net at R?.1: now also VT?.2 (x2)
- net at R24.1: now also VT?.3
- net at R?.2, U10.12: now also VT?.3
- net at R?.1: now also VT1.1, VT15.2
- net at R45.2: now also VT1.2
- net at D?.1 (K), J?.1 (Pin_1): now also VT1.3, VT15.3
- net at R?.1: now also VT16.2, VT2.1
- net at R46.2: now also VT2.2
- net at D?.1 (K), J?.2 (Pin_2): now also VT16.3, VT2.3
- net at R?.1: now also VT.1, VT17.2
- net at R47.2: now also VT.2
- net at D?.1 (K), J?.3 (Pin_3): now also VT.3, VT17.3
- net at R?.1: now also VT18.2, VT4.1
- net at R48.2: now also VT4.2
- net at D?.1 (K), J?.4 (Pin_4): now also VT18.3, VT4.3
- net at R?.1: now also VT19.2, VT7.1
- net at R?.2: now also VT7.2
- net at D?.1 (K), J?.1 (Pin_1): now also VT19.3, VT7.3
- net at R?.1: now also VT20.2, VT8.1
- net at R?.2: now also VT8.2
- net at D?.1 (K), J?.2 (Pin_2): now also VT20.3, VT8.3
- net at R?.1: now also VT21.2, VT9.1
- net at R?.2: now also VT9.2
- net at D?.1 (K), J?.3 (Pin_3): now also VT21.3, VT9.3
- net at R?.1: now also VT10.1, VT22.2
- net at R?.2: now also VT10.2
- net at D?.1 (K), J?.4 (Pin_4): now also VT10.3, VT22.3
- net at R49.2: now also VT5.2
- net at R?.2: now also VT5.3
- net at R?.1, R?.2: now also VT26.3
- net at D?.1 (K), D?.2 (A), J?.5 (Pin_5): now also VT26.2
- net at R50.2: now also VT6.2
- net at R?.2: now also VT6.3
- net at R?.1, R?.2: now also VT27.3
- net at D?.1 (K), D?.2 (A), J?.6 (Pin_6): now also VT27.2
- net at R?.2: now also VT11.2
- net at R?.2: now also VT11.3
- net at R?.1, R?.2: now also VT28.3
- net at D?.1 (K), D?.2 (A), J?.5 (Pin_5): now also VT28.2
- net at R?.2: now also VT12.2
- net at R?.2: now also VT12.3
- net at R?.1, R?.2: now also VT29.3
- net at D?.1 (K), D?.2 (A), J?.6 (Pin_6): now also VT29.2
