File: kicad/xy4150.sch (KiCad schematic (older format))
At the start: 200 parts, among them J1 PEN, J10 MG, J11 MG, J12 MG, J13 MG, J14 MG, J15 MG, J16 Conn_01x06, J17 Conn_01x06, J2 LD, J3 LD, J4 PD, J5 LD, J6 +/-, J7 X/Y, J8 /MOV, J9 /RDY, U1 4011, U10 7403, U11 4001, U12 4001, U13 4013, U14 4069, U15 4001, U16 L7805, U2 4011, U3 4029, U4 4029, U5 4069, U6 4001, U7 4012, U8 4030, U9 4001

Commit message: update pcb
Parts:
- R1, R64: value R -> 3k9
- R12: value R -> 100R
- R26: value R -> 220R
- R31: value R -> 15k
- R5: value R -> 3.9k
- R52, R55, R69: value R -> 1k8
Connections:
- net Vcc is gone; now on net +5V: U10.14 (Vcc), U10.14 (Vcc), U10.14 (Vcc), U10.14 (Vcc)
- net Vdd is gone; now on net GND: U8.14 (Vdd), U8.14 (Vdd), U8.14 (Vdd), U8.14 (Vdd)
- net Vss is gone; now on net GND: U8.7 (Vss), U8.7 (Vss), U8.7 (Vss), U8.7 (Vss)
- net +5V: no longer D10.2 (A), J10.1 (Pin_1), VT23.1
- net at D6.2 (A), R41.1, U11.12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: no longer U12.6
- new net: D10.2 (A), J10.1 (Pin_1), VT23.1
Changed lines of the file:
@@
 P -3200 -3800
 F 0 "R1" H -3130 -3754 50  0000 L CNN
-F 1 "R" H -3130 -3845 50  0000 L CNN
+F 1 "3k9" H -3130 -3845 50  0000 L CNN
 F 2 "Resistor_THT:R_Axial_DIN0207_L6.3mm_D2.5mm_P10.16mm_Horizontal" V -3270 -3800 50  0001 C CNN
 F 3 "~" H -3200 -3800 50  0001 C CNN
@@
 $EndComp
 Wire Wire Line
-	6450 -1600 6400 -1600
-Wire Wire Line
 	5750 -2150 4650 -2150
-Connection ~ 6400 -1600
-Wire Wire Line
-	6400 -1600 5750 -1600
 Connection ~ 4650 -3100
 Wire Wire Line
@@
 P -3650 -2550
 F 0 "R12" V -3600 -2750 50  0000 C CNN
-F 1 "R" V -3500 -2750 50  0000 C CNN
+F 1 "100R" V -3500 -2750 50  0000 C CNN
 F 2 "Resistor_THT:R_Axial_DIN0207_L6.3mm_D2.5mm_P10.16mm_Horizontal" V -3720 -2550 50  0001 C CNN
 F 3 "~" H -3650 -2550 50  0001 C CNN
@@
 P -4050 -2000
 F 0 "R5" H -3980 -1954 50  0000 L CNN
-F 1 "R" H -3980 -2045 50  0000 L CNN
+F 1 "3.9k" H -3980 -2045 50  0000 L CNN
 F 2 "Resistor_THT:R_Axial_DIN0207_L6.3mm_D2.5mm_P10.16mm_Horizontal" V -4120 -2000 50  0001 C CNN
 F 3 "~" H -4050 -2000 50  0001 C CNN
@@
 P 100 4900
 F 0 "R31" V -107 4900 50  0000 C CNN
-F 1 "R" V -16 4900 50  0000 C CNN
+F 1 "15k" V -16 4900 50  0000 C CNN
 F 2 "Resistor_THT:R_Axial_DIN0207_L6.3mm_D2.5mm_P10.16mm_Horizontal" V 30  4900 50  0001 C CNN
 F 3 "~" H 100 4900 50  0001 C CNN
@@
 Wire Wire Line
 	1550 4650 1550 4750
-Wire Wire Line
-	1950 4650 1950 4750
 Connection ~ 1950 4650
 Wire Wire Line
@@
 	1550 5150 1550 5050
 $Comp
-L power:+5V #PWR0136
-U 1 1 5F80D078
-P 1950 4550
-F 0 "#PWR0136" H 1950 4400 50  0001 C CNN
-F 1 "+5V" H 1965 4723 50  0000 C CNN
-F 2 "" H 1950 4550 50  0001 C CNN
-F 3 "" H 1950 4550 50  0001 C CNN
-	1    1950 4550
-	1    0    0    -1
-$EndComp
-Wire Wire Line
-	1950 4550 1950 4650
-$Comp
 L Device:R R34
 U 1 1 5F842C12
@@
 P 3500 4900
 F 0 "R26" H 3570 4946 50  0000 L CNN
-F 1 "R" H 3570 4855 50  0000 L CNN
+F 1 "220R" H 3570 4855 50  0000 L CNN
 F 2 "Resistor_THT:R_Axial_DIN0207_L6.3mm_D2.5mm_P10.16mm_Horizontal" V 3430 4900 50  0001 C CNN
 F 3 "~" H 3500 4900 50  0001 C CNN
@@
 	-350 3250 -350 4550
 Wire Wire Line
-	-350 4550 1950 4550
-Wire Wire Line
 	4250 4550 4250 4650
-Connection ~ 1950 4550
-Wire Wire Line
-	1950 4550 4250 4550
 Connection ~ 4250 4650
 Wire Wire Line
@@
 P 7950 -1050
 F 0 "R52" H 7750 -1000 50  0000 L CNN
-F 1 "R" H 7750 -1100 50  0000 L CNN
+F 1 "1k8" H 7750 -1100 50  0000 L CNN
 F 2 "Resistor_THT:R_Axial_DIN0207_L6.3mm_D2.5mm_P10.16mm_Horizontal" V 7880 -1050 50  0001 C CNN
 F 3 "~" H 7950 -1050 50  0001 C CNN
@@
 P 9250 -1050
 F 0 "R55" H 9050 -1000 50  0000 L CNN
-F 1 "R" H 9050 -1100 50  0000 L CNN
+F 1 "1k8" H 9050 -1100 50  0000 L CNN
 F 2 "Resistor_THT:R_Axial_DIN0207_L6.3mm_D2.5mm_P10.16mm_Horizontal" V 9180 -1050 50  0001 C CNN
 F 3 "~" H 9250 -1050 50  0001 C CNN
@@
 P 13300 -1050
 F 0 "R64" H 13100 -1000 50  0000 L CNN
-F 1 "R" H 13100 -1100 50  0000 L CNN
+F 1 "3k9" H 13100 -1100 50  0000 L CNN
 F 2 "Resistor_THT:R_Axial_DIN0207_L6.3mm_D2.5mm_P10.16mm_Horizontal" V 13230 -1050 50  0001 C CNN
 F 3 "~" H 13300 -1050 50  0001 C CNN
@@
 P 15500 -1050
 F 0 "R69" H 15300 -1000 50  0000 L CNN
-F 1 "R" H 15300 -1100 50  0000 L CNN
+F 1 "1k8" H 15300 -1100 50  0000 L CNN
 F 2 "Resistor_THT:R_Axial_DIN0207_L6.3mm_D2.5mm_P10.16mm_Horizontal" V 15430 -1050 50  0001 C CNN
 F 3 "~" H 15500 -1050 50  0001 C CNN
@@
 	19800 2450 19200 2450
 Wire Wire Line
-	8200 3300 8300 3300
-$Comp
-L power:PWR_FLAG #FLG04
-U 1 1 67F786BF
-P 8200 3300
-F 0 "#FLG04" H 8200 3375 50  0001 C CNN
-F 1 "PWR_FLAG" H 8200 3473 50  0000 C CNN
-F 2 "" H 8200 3300 50  0001 C CNN
-F 3 "~" H 8200 3300 50  0001 C CNN
-	1    8200 3300
-	1    0    0    -1
-$EndComp
-Wire Wire Line
-	8200 2800 8300 2800
-$Comp
-L power:PWR_FLAG #FLG03
-U 1 1 67F78167
-P 8200 2800
-F 0 "#FLG03" H 8200 2875 50  0001 C CNN
-F 1 "PWR_FLAG" H 8200 2973 50  0000 C CNN
-F 2 "" H 8200 2800 50  0001 C CNN
-F 3 "~" H 8200 2800 50  0001 C CNN
-	1    8200 2800
-	1    0    0    -1
-$EndComp
-Wire Wire Line
-	8200 2200 8300 2200
-$Comp
-L power:PWR_FLAG #FLG02
-U 1 1 67F77C98
-P 8200 2200
-F 0 "#FLG02" H 8200 2275 50  0001 C CNN
-F 1 "PWR_FLAG" H 8200 2373 50  0000 C CNN
-F 2 "" H 8200 2200 50  0001 C CNN
-F 3 "~" H 8200 2200 50  0001 C CNN
-	1    8200 2200
-	1    0    0    -1
-$EndComp
-Wire Wire Line
-	8200 1700 8300 1700
-$Comp
-L power:PWR_FLAG #FLG01
-U 1 1 67F75237
-P 8200 1700
-F 0 "#FLG01" H 8200 1775 50  0001 C CNN
-F 1 "PWR_FLAG" H 8200 1873 50  0000 C CNN
-F 2 "" H 8200 1700 50  0001 C CNN
-F 3 "~" H 8200 1700 50  0001 C CNN
-	1    8200 1700
-	1    0    0    -1
-$EndComp
-Wire Wire Line
 	8950 2650 8950 3150
 Wire Wire Line
@@
 Wire Wire Line
 	8300 3300 8300 3150
-Connection ~ 8200 3300
-Wire Wire Line
-	8150 3300 8200 3300
 Wire Wire Line
 	8300 2950 8400 2950
@@
 Wire Wire Line
 	8300 2800 8300 2650
-Connection ~ 8200 2800
-Wire Wire Line
-	8150 2800 8200 2800
 Wire Wire Line
 	8300 2350 8400 2350
@@
 Wire Wire Line
 	8300 2200 8300 2050
-Connection ~ 8200 2200
-Wire Wire Line
-	8150 2200 8200 2200
 Wire Wire Line
 	8300 1850 8400 1850
@@
 Wire Wire Line
 	8300 1700 8300 1550
-Connection ~ 8200 1700
-Wire Wire Line
-	8150 1700 8200 1700
 $Comp
 L Connector:Conn_01x01_Female J15
@@
 	1    0    0    -1
 $EndComp
+$Comp
+L power:GND #PWR0165
+U 1 1 5DA210AD
+P 1650 3350
+F 0 "#PWR0165" H 1650 3100 50  0001 C CNN
+F 1 "GND" H 1655 3177 50  0000 C CNN
+F 2 "" H 1650 3350 50  0001 C CNN
+F 3 "" H 1650 3350 50  0001 C CNN
+	1    1650 3350
+	1    0    0    -1
+$EndComp
+$Comp
+L power:+5V #PWR0168
+U 1 1 5DA25038
+P 1650 2850
+F 0 "#PWR0168" H 1650 2700 50  0001 C CNN
+F 1 "+5V" H 1665 3023 50  0000 C CNN
+F 2 "" H 1650 2850 50  0001 C CNN
+F 3 "" H 1650 2850 50  0001 C CNN
+	1    1650 2850
+	1    0    0    -1
+$EndComp
+$Comp
+L power:GND #PWR0170
+U 1 1 5DA362F2
+P 1650 4300
+F 0 "#PWR0170" H 1650 4050 50  0001 C CNN
+F 1 "GND" H 1655 4127 50  0000 C CNN
+F 2 "" H 1650 4300 50  0001 C CNN
+F 3 "" H 1650 4300 50  0001 C CNN
+	1    1650 4300
+	1    0    0    -1
+$EndComp
+$Comp
+L power:+5V #PWR0171
+U 1 1 5DA36968
+P 1650 3800
+F 0 "#PWR0171" H 1650 3650 50  0001 C CNN
+F 1 "+5V" H 1665 3973 50  0000 C CNN
+F 2 "" H 1650 3800 50  0001 C CNN
+F 3 "" H 1650 3800 50  0001 C CNN
+	1    1650 3800
+	1    0    0    -1
+$EndComp
+$Comp
+L power:GND #PWR0173
+U 1 1 5DA416BF
+P 5450 2100
+F 0 "#PWR0173" H 5450 1850 50  0001 C CNN
+F 1 "GND" H 5455 1927 50  0000 C CNN
+F 2 "" H 5450 2100 50  0001 C CNN
+F 3 "" H 5450 2100 50  0001 C CNN
+	1    5450 2100
+	1    0    0    -1
+$EndComp
+$Comp
+L power:GND #PWR0172
+U 1 1 5DA5EFA7
+P 5450 -2200
+F 0 "#PWR0172" H 5450 -2450 50  0001 C CNN
+F 1 "GND" H 5455 -2373 50  0000 C CNN
+F 2 "" H 5450 -2200 50  0001 C CNN
+F 3 "" H 5450 -2200 50  0001 C CNN
+	1    5450 -2200
+	1    0    0    -1
+$EndComp
+$Comp
+L power:GND #PWR0174
+U 1 1 5DA7158B
+P 3850 -2500
+F 0 "#PWR0174" H 3850 -2750 50  0001 C CNN
+F 1 "GND" H 3855 -2673 50  0000 C CNN
+F 2 "" H 3850 -2500 50  0001 C CNN
+F 3 "" H 3850 -2500 50  0001 C CNN
+	1    3850 -2500
+	1    0    0    -1
+$EndComp
+$Comp
+L power:GND #PWR0175
+U 1 1 5DA792E6
+P 3850 1800
+F 0 "#PWR0175" H 3850 1550 50  0001 C CNN
+F 1 "GND" H 3855 1627 50  0000 C CNN
+F 2 "" H 3850 1800 50  0001 C CNN
+F 3 "" H 3850 1800 50  0001 C CNN
+	1    3850 1800
+	1    0    0    -1
+$EndComp
+$Comp
+L power:GND #PWR0176
+U 1 1 5DA7EEB1
+P 2950 3650
+F 0 "#PWR0176" H 2950 3400 50  0001 C CNN
+F 1 "GND" H 2955 3477 50  0000 C CNN
+F 2 "" H 2950 3650 50  0001 C CNN
+F 3 "" H 2950 3650 50  0001 C CNN
+	1    2950 3650
+	1    0    0    -1
+$EndComp
+$Comp
+L power:GND #PWR0177
+U 1 1 5DA7F5F9
+P 2950 4200
+F 0 "#PWR0177" H 2950 3950 50  0001 C CNN
+F 1 "GND" H 2955 4027 50  0000 C CNN
+F 2 "" H 2950 4200 50  0001 C CNN
+F 3 "" H 2950 4200 50  0001 C CNN
+	1    2950 4200
+	1    0    0    -1
+$EndComp
+Wire Wire Line
+	5750 -1600 6450 -1600
+Wire Wire Line
+	8150 1700 8300 1700
+Wire Wire Line
+	8150 2200 8300 2200
+Wire Wire Line
+	8150 2800 8300 2800
+Wire Wire Line
+	8150 3300 8300 3300
+Wire Wire Line
+	-350 4550 4250 4550
+Wire Wire Line
+	1950 4650 1950 4750
+$Comp
+L power:+5V #PWR0136
+U 1 1 5F80D078
+P 1950 4650
+F 0 "#PWR0136" H 1950 4500 50  0001 C CNN
+F 1 "+5V" H 1965 4823 50  0000 C CNN
+F 2 "" H 1950 4650 50  0001 C CNN
+F 3 "" H 1950 4650 50  0001 C CNN
+	1    1950 4650
+	1    0    0    -1
+$EndComp

Commit message: update pcb
Parts:
- removed VT15, VT16, VT17, VT18, VT19, VT20, VT21, VT22, VT23, VT3: KC639, Package_TO_SOT_THT:TO-92, symbol xy4150-restore:KC639
- added VT15, VT16, VT17, VT18, VT19, VT20, VT21, VT22, VT23: KD139, Package_TO_SOT_THT:TO-126-3_Vertical, symbol xy4150-restore:KD139
- added VT3: KC636, Package_TO_SOT_THT:TO-92, symbol xy4150-restore:KC636
- C5: value C -> 6n; footprint Capacitor_THT:C_Disc_D10.0mm_W2.5mm_P5.00mm -> Capacitor_THT:C_Disc_D7.5mm_W2.5mm_P5.00mm
- C6: value C -> 1u (TC205); footprint Capacitor_THT:C_Disc_D10.0mm_W2.5mm_P5.00mm -> Capacitor_THT:C_Axial_L19.0mm_D9.5mm_P25.00mm_Horizontal
- R10, R11, R14: value R -> 100R
- R15: value R -> 180k
- R17: value R -> 150k
- R2, R21, R6, R7: value R -> 3k9
- R22, R28, R32: value R -> 27k
- R27, R34: value R -> 15k
- R33: value R -> 220R
- R36: value R -> 4k7
- R45, R46, R47, R48, R49, R50, R58, R61: value R -> 1k8
- R53, R54, R56, R57, R59, R60, R62, R63, R67, R68, R72, R73: value R -> 820R
- R64: value 3k9 -> 1k8
- R65, R66, R70, R71: value R -> 1k5
Connections:
- net +5V: now also VT3.3
- net GND: now also C6.2, D2.1 (K), R27.2, R30.2, R37.2, VT13.3, VT15.1, VT16.1, VT17.1, VT18.1, VT19.1, VT20.1, VT21.1, VT22.1
- net at R32.1: now also VT3.2
- net at R21.2: now also VT3.1
- net at C7.2, D1.2 (A), R29.1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: now also VT23.1
- net at R37.1, VT14.3: now also VT23.3
- net at D10.2 (A), J10.1 (Pin_1): now also VT23.2
- net at R53.1, VT1.3: now also VT15.3
- net at D19.1 (K), J16.1 (Pin_1), VT1.1: now also VT15.2
- net at R56.1, VT2.3: now also VT17.3
- net at D21.1 (K), J16.2 (Pin_2), VT2.1: now also VT17.2
- net at R59.1, VT30.3: now also VT19.3
- net at D23.1 (K), J16.3 (Pin_3), VT30.1: now also VT19.2
- net at R62.1, VT4.3: now also VT21.3
- net at D25.1 (K), J16.4 (Pin_4), VT4.1: now also VT21.2
- net at R54.1, VT7.3: now also VT16.3
- net at D20.1 (K), J17.1 (Pin_1), VT7.1: now also VT16.2
- net at R57.1, VT8.3: now also VT18.3
- net at D22.1 (K), J17.2 (Pin_2), VT8.1: now also VT18.2
- net at R60.1, VT9.3: now also VT20.3
- net at D24.1 (K), J17.3 (Pin_3), VT9.1: now also VT20.2
- net at R63.1, VT10.3: now also VT22.3
- net at D26.1 (K), J17.4 (Pin_4), VT10.1: now also VT22.2

Commit message: update pcb and schema
Parts:
- added unit 3 of U13
- C13: footprint Capacitor_THT:C_Disc_D10.0mm_W2.5mm_P5.00mm -> xy4150-restore:TE-61x25
- C14: value C -> 5m (TE674); footprint Capacitor_THT:C_Disc_D10.0mm_W2.5mm_P5.00mm -> xy4150-restore:TE-61x25
- R19, R20: value R -> 180R
- R24: value R -> 220R
- R25, R51: value R -> 27k
- R3: value R -> 3k9
- R39, R40: value R -> 2k2
Connections:
- net +5V: now also U12.14 (VDD), U15.14 (VDD), U13.14 (VDD); no longer U10.14 (Vcc), U10.14 (Vcc), U10.14 (Vcc), U10.14 (Vcc), U12.7 (VSS), U15.7 (VSS)
- net GND: now also C13.2, U12.7 (VSS), U15.7 (VSS), U13.7 (VSS); no longer C13.1, U12.14 (VDD), U15.14 (VDD)
- net at D6.2 (A), R41.1, U11.12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: now also U12.6
- net at U2.3, U7.10: now also U7.5; no longer U7.3
- net at C1.1, R13.2: now also U7.3; no longer U7.5
- net at D16.1 (K), D18.1 (K), JP5.1 (A)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: now also C13.1; no longer C13.2
- new net Vcc: U10.14 (Vcc), U10.14 (Vcc), U10.14 (Vcc), U10.14 (Vcc)
Other:
- moved on the sheet: C1, C10, C11, C12, C13, C14, C15, C16, C17, C18, C19, C2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
