File: kicad/xy4150.kicad_pcb (KiCad board)
At the start: 2 copper layers, 200 parts, among them J1 PEN, J10 MG, J11 MG, J12 MG, J13 MG, J14 MG, J15 MG, J16 Conn_01x06, J17 Conn_01x06, J2 LD, J3 LD, J4 PD, J5 LD, J6 +/-, J7 X/Y, J8 /MOV, J9 /RDY, U1 4011, U10 7403, U11 4001, U12 4001, U13 4013, U14 4069, U15 4001, U16 L7805, U2 4011, U3 4029, U4 4029, U5 4069, U6 4001, U7 4012, U8 4030, U9 4001

Commit message: update pcb
Parts:
- R1, R64: value R -> 3k9
- R12: value R -> 100R
- R26: value R -> 220R
- R31: value R -> 15k
- R45, R46, R47, R48, R52, R55, R58, R61, R69: value R -> 1k8
- R5: value R -> 3.9k
- moved J7 258.1 mm to (127.0, -52.1)
- moved R1 160.9 mm to (132.1, 19.1), turned to 90 degrees
- moved R12 148.8 mm to (132.1, 7.62), turned to 90 degrees
- moved R52 117.9 mm to (218.4, 10.2)
- moved R69 109.0 mm to (218.4, 39.4)
- moved R26 104.8 mm to (218.4, 6.35)
- moved R64 84.8 mm to (218.4, 31.8)
- moved R31 72.7 mm to (228.6, 41.9), turned to 180 degrees
- moved R7 40.0 mm to (248.9, 19.1), turned to 180 degrees
- moved U8 17.0 mm to (180.3, 19.1), turned to 180 degrees
Connections:
- D10 pad 2: +5V -> Net-(D10-Pad2)
- J10 pad 1: +5V -> Net-(D10-Pad2)
- U10 pad 14: (no net) -> +5V
- U12 pad 6: Net-(D6-Pad2) -> (no net)
- U8 pad 14: (no net) -> GND
- U8 pad 7: (no net) -> GND
- VT23 pad 3: +5V -> Net-(D10-Pad2)
Routing:
- net GND: track 0.00 -> 166.4 mm, vias 0 -> 1
- net (no net): track 0.00 -> 131.9 mm, vias 1 -> 9
- net /m2-1: track 0.00 -> 115.6 mm
- net Net-(R1-Pad2): track 0.00 -> 102.7 mm, vias 0 -> 1
- net +5V: track 95.0 -> 178.9 mm
- net Net-(U1-Pad2): track 0.00 -> 69.8 mm, vias 0 -> 2
- net Net-(R31-Pad2): track 0.00 -> 68.6 mm
- net Net-(U3-Pad11): track 0.00 -> 44.5 mm, vias 0 -> 1
- net Net-(U11-Pad6): track 0.00 -> 43.7 mm
- net Net-(U14-Pad12): track 0.00 -> 29.2 mm
- net Net-(U14-Pad3): track 0.00 -> 26.7 mm, vias 0 -> 1
- net Net-(U4-Pad11): track 0.00 -> 24.1 mm, vias 0 -> 1
- net Net-(U2-Pad12): track 0.00 -> 21.6 mm, vias 0 -> 1
- net Net-(U5-Pad4): track 0.00 -> 14.0 mm, vias 0 -> 1
- net Net-(U6-Pad11): track 0.00 -> 12.7 mm
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
Commit message: update pcb
Parts:
- C5: value C -> 6n; footprint Capacitor_THT:C_Disc_D10.0mm_W2.5mm_P5.00mm -> Capacitor_THT:C_Disc_D7.5mm_W2.5mm_P5.00mm
- C6: value C -> 1u (TC205); footprint Capacitor_THT:C_Disc_D10.0mm_W2.5mm_P5.00mm -> Capacitor_THT:C_Axial_L19.0mm_D9.5mm_P25.00mm_Horizontal
- R10, R11, R14: value R -> 100R
- R15: value R -> 180k
- R17: value R -> 150k
- R2, R21, R6, R7: value R -> 3k9
- R22, R28, R32: value R -> 27k
- R27, R34: value R -> 15k
- R33: value R -> 220R
- R36: value R -> 4k7
- R49, R50: value R -> 1k8
- R53, R54, R56, R57, R59, R60, R62, R63, R67, R68, R72, R73: value R -> 820R
- R64: value 3k9 -> 1k8
- R65, R66, R70, R71: value R -> 1k5
- VT15, VT16, VT17, VT18, VT19, VT20, VT21, VT22, VT23: value KC639 -> KD139; footprint Package_TO_SOT_THT:TO-92 -> Package_TO_SOT_THT:TO-126-3_Vertical
- VT3: value KC639 -> KC636
- moved J11 285.9 mm to (96.5, -57.1)
- moved VT15 280.2 mm to (101.6, -39.4), turned to 270 degrees
- moved VT1 276.3 mm to (111.8, -38.1), turned to 270 degrees
- moved R71 271.2 mm to (82.5, 57.1)
- moved R41 270.4 mm to (96.5, 82.5), turned to 180 degrees
- moved J3 268.8 mm to (114.3, -57.1)
- moved VT17 260.9 mm to (101.6, -26.7), turned to 270 degrees
- moved VT4 258.4 mm to (111.8, 7.62), turned to 270 degrees
- moved J6 255.9 mm to (134.6, -59.7)
- moved J8 253.6 mm to (141.0, -63.5)
- moved D19 251.5 mm to (97.8, -31.8), turned to 90 degrees
- moved VT6 250.5 mm to (88.9, 61.0), turned to 180 degrees
- moved J1 250.4 mm to (146.1, -58.4)
- moved VT2 243.9 mm to (111.8, -25.4), turned to 270 degrees
- moved C9 243.8 mm to (110.5, 82.5)
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Connections:
- C6 pad 2: Net-(C6-Pad2) -> GND
- D2 pad 1: Net-(C6-Pad2) -> GND
- R27 pad 2: Net-(C6-Pad2) -> GND
- R30 pad 2: Net-(C6-Pad2) -> GND
- R37 pad 2: Net-(C6-Pad2) -> GND
- VT1 pad 1: Net-(R53-Pad1) -> Net-(D19-Pad1)
- VT1 pad 3: Net-(D19-Pad1) -> Net-(R53-Pad1)
- VT10 pad 1: Net-(R63-Pad1) -> Net-(D26-Pad1)
- VT10 pad 3: Net-(D26-Pad1) -> Net-(R63-Pad1)
- VT11 pad 1: GND -> Net-(R65-Pad2)
- VT11 pad 3: Net-(R65-Pad2) -> GND
- VT12 pad 1: GND -> Net-(R70-Pad2)
- VT12 pad 3: Net-(R70-Pad2) -> GND
- VT13 pad 1: Net-(C6-Pad2) -> Net-(C5-Pad1)
- VT13 pad 3: Net-(C5-Pad1) -> GND
- VT14 pad 1: Net-(R37-Pad1) -> Net-(R33-Pad1)
- VT14 pad 3: Net-(R33-Pad1) -> Net-(R37-Pad1)
- VT15 pad 2: Net-(R53-Pad1) -> Net-(D19-Pad1)
- VT15 pad 3: Net-(D19-Pad1) -> Net-(R53-Pad1)
- VT16 pad 2: Net-(R56-Pad1) -> Net-(D20-Pad1)
- VT16 pad 3: Net-(D21-Pad1) -> Net-(R54-Pad1)
- VT17 pad 2: Net-(R59-Pad1) -> Net-(D21-Pad1)
- VT17 pad 3: Net-(D23-Pad1) -> Net-(R56-Pad1)
- VT18 pad 2: Net-(R62-Pad1) -> Net-(D22-Pad1)
- VT18 pad 3: Net-(D25-Pad1) -> Net-(R57-Pad1)
- VT19 pad 2: Net-(R54-Pad1) -> Net-(D23-Pad1)
- VT19 pad 3: Net-(D20-Pad1) -> Net-(R59-Pad1)
- VT2 pad 1: Net-(R56-Pad1) -> Net-(D21-Pad1)
- VT2 pad 3: Net-(D21-Pad1) -> Net-(R56-Pad1)
- VT20 pad 2: Net-(R57-Pad1) -> Net-(D24-Pad1)
- VT20 pad 3: Net-(D22-Pad1) -> Net-(R60-Pad1)
- VT21 pad 2: Net-(R60-Pad1) -> Net-(D25-Pad1)
- VT21 pad 3: Net-(D24-Pad1) -> Net-(R62-Pad1)
- VT22 pad 2: Net-(R63-Pad1) -> Net-(D26-Pad1)
- VT22 pad 3: Net-(D26-Pad1) -> Net-(R63-Pad1)
- VT23 pad 2: Net-(R37-Pad1) -> Net-(D10-Pad2)
- VT23 pad 3: Net-(D10-Pad2) -> Net-(R37-Pad1)
- VT24 pad 1: GND -> Net-(R24-Pad1)
- VT24 pad 3: Net-(R24-Pad1) -> GND
- VT25 pad 1: GND -> Net-(R36-Pad2)
- VT25 pad 3: Net-(R36-Pad2) -> GND
- VT30 pad 1: Net-(R59-Pad1) -> Net-(D23-Pad1)
- VT30 pad 3: Net-(D23-Pad1) -> Net-(R59-Pad1)
- VT4 pad 1: Net-(R62-Pad1) -> Net-(D25-Pad1)
- VT4 pad 3: Net-(D25-Pad1) -> Net-(R62-Pad1)
- VT5 pad 1: GND -> Net-(R66-Pad2)
- VT5 pad 3: Net-(R66-Pad2) -> GND
- VT6 pad 1: GND -> Net-(R71-Pad2)
- VT6 pad 3: Net-(R71-Pad2) -> GND
- VT7 pad 1: Net-(R54-Pad1) -> Net-(D20-Pad1)
- VT7 pad 3: Net-(D20-Pad1) -> Net-(R54-Pad1)
- VT8 pad 1: Net-(R57-Pad1) -> Net-(D22-Pad1)
- VT8 pad 3: Net-(D22-Pad1) -> Net-(R57-Pad1)
- VT9 pad 1: Net-(R60-Pad1) -> Net-(D24-Pad1)
- VT9 pad 3: Net-(D24-Pad1) -> Net-(R60-Pad1)
Routing:
- net (no net): track 131.9 -> 585.0 mm, vias 9 -> 14
- net GND: track 166.4 -> 418.5 mm
- net +5V: track 178.9 -> 356.2 mm, vias 0 -> 2
- net Net-(D9-Pad2): track 0.00 -> 149.5 mm
- net Net-(R34-Pad2): track 0.00 -> 144.8 mm, vias 0 -> 1
- net Net-(C10-Pad1): track 0.00 -> 116.4 mm
- net Net-(C4-Pad1): track 0.00 -> 110.4 mm, vias 0 -> 1
- net +24V: track 0.00 -> 108.5 mm
- net Net-(D5-Pad1): track 0.00 -> 107.9 mm
- net /m1-1: track 0.00 -> 101.9 mm
- net /m2-2: track 0.00 -> 99.1 mm, vias 0 -> 1
- net Net-(D8-Pad2): track 0.00 -> 93.9 mm
- net Net-(D20-Pad1): track 0.00 -> 83.8 mm
- net /m1-3: track 0.00 -> 83.8 mm
- net /m1-4: track 0.00 -> 81.3 mm
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
Commit message: update pcb and schema
Parts:
- C13: footprint Capacitor_THT:C_Disc_D10.0mm_W2.5mm_P5.00mm -> xy4150-restore:TE-61x25
- C14: value C -> 5m (TE674); footprint Capacitor_THT:C_Disc_D10.0mm_W2.5mm_P5.00mm -> xy4150-restore:TE-61x25
- R19, R20: value R -> 180R
- R24: value R -> 220R
- R25, R51: value R -> 27k
- R3: value R -> 3k9
- R40: value R -> 2k2
- moved J5 270.6 mm to (121.9, -57.1)
- moved J4 266.0 mm to (130.8, -62.2)
- moved J9 239.2 mm to (151.1, -68.6)
- moved D10 178.5 mm to (162.6, -39.4), turned to 180 degrees
- moved R35 170.9 mm to (398.8, 54.6), turned to 270 degrees
- moved D17 148.8 mm to (330.2, 90.2), turned to 270 degrees
- moved D16 146.7 mm to (337.8, 100.3), turned to 90 degrees
- moved D7 143.5 mm to (219.7, 109.2)
- moved C12 142.1 mm to (294.6, 82.5), turned to 90 degrees
- moved D15 142.0 mm to (334.0, 90.2), turned to 270 degrees
- moved D12 137.7 mm to (318.8, 74.9), turned to 180 degrees
- moved D18 135.6 mm to (326.4, 100.3), turned to 90 degrees
- moved J14 134.3 mm to (332.7, 81.3), turned to 90 degrees
- moved J15 133.3 mm to (336.6, 81.3), turned to 90 degrees
- moved R44 132.5 mm to (318.8, -10.2), turned to 180 degrees
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Connections:
- C13 pad 1: GND -> Net-(C13-Pad1)
- C13 pad 2: Net-(C13-Pad2) -> GND
- D16 pad 1: Net-(C13-Pad2) -> Net-(C13-Pad1)
- D18 pad 1: Net-(C13-Pad2) -> Net-(C13-Pad1)
- JP5 pad 1: Net-(C13-Pad2) -> Net-(C13-Pad1)
- JP6 pad 1: Net-(C13-Pad2) -> Net-(C13-Pad1)
- U10 pad 14: +5V -> (no net)
- U12 pad 14: GND -> +5V
- U12 pad 6: (no net) -> Net-(D6-Pad2)
- U12 pad 7: +5V -> GND
- U13 pad 14: (no net) -> +5V
- U13 pad 7: (no net) -> GND
- U15 pad 14: GND -> +5V
- U15 pad 7: +5V -> GND
- U7 pad 3: Net-(U2-Pad3) -> Net-(C1-Pad1)
- U7 pad 5: Net-(C1-Pad1) -> Net-(U2-Pad3)
Routing:
- net (no net): track 585.0 -> 870.4 mm, vias 14 -> 13
- net +24V: track 108.5 -> 379.0 mm, vias 0 -> 1
- net GND: track 418.5 -> 631.9 mm, vias 1 -> 5
- net Net-(C11-Pad2): track 0.00 -> 188.4 mm, vias 0 -> 2
- net Net-(D8-Pad2): track 93.9 -> 256.4 mm
- net Net-(D5-Pad1): track 107.9 -> 264.2 mm, vias 0 -> 2
- net Net-(D10-Pad2): track 0.00 -> 128.3 mm
- net Net-(D9-Pad2): track 149.5 -> 272.7 mm
- net Net-(R3-Pad2): track 0.00 -> 121.9 mm
- net Net-(R31-Pad1): track 67.1 -> 159.1 mm, vias 0 -> 1
- net Net-(R29-Pad2): track 0.00 -> 87.0 mm
- net Net-(C10-Pad1): track 116.4 -> 181.2 mm
- net Net-(C7-Pad2): track 0.00 -> 59.7 mm
- net Net-(D7-Pad2): track 31.0 -> 89.4 mm, vias 1 -> 2
- net +5V: track 356.2 -> 303.4 mm, vias 2 -> 3
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